File: TICK/TICK_AC/TICK_AC.sch (KiCad schematic (older format))
At the start: 8 parts, among them CN1 To_Amiga, CN2 Barrel_Jack_MountingPin, U1 74AHCT1G04

Commit message: Add files via upload
Parts:
- removed C2: 0.1uF, Capacitor_SMD:C_1206_3216Metric, symbol Device:C
- removed U1: 74AHCT1G04, Package_TO_SOT_SMD:SOT-23-5, symbol 74xGxx:SN74LVC1G14DBV
- added Q1: MMBT3904, Package_TO_SOT_SMD:SOT-23, symbol Transistor_BJT:MMBT3904
- C1: value 22uF -> 0.22uF
- CN2: value Barrel_Jack_MountingPin -> Barrel_Jack; footprint Connector_BarrelJack:BarrelJack_CUI_PJ-102AH_Horizontal -> TICK:BarrelJack_Horizontal; symbol Connector:Barrel_Jack_MountingPin -> Connector:Barrel_Jack
- D1: value MMSZ5225 -> 1N4148; symbol Device:D_Zener -> Device:D
- R1: value 560 -> 3.3k
- R2: value 10k -> 4.7k
Connections:
- net +5V: now also R2.2; no longer R2.1
- net GND: now also Q1.2 (E); no longer CN2.MP (MountPin)
- net TBASE: now also R2.1, Q1.3 (C); no longer R2.2
- net at C1.1, D1.1 (K), R1.1: now also Q1.1 (B)
Other:
- note removed: "D1 = 3V, 500mw"
- moved on the sheet: C1, CN1, D1
Changed lines of the file:
@@
 L Connector:Conn_01x06_Female CN1
 U 1 1 61AA2F62
-P 6750 3200
-F 0 "CN1" H 6778 3176 50  0000 L CNN
-F 1 "To_Amiga" H 6778 3085 50  0000 L CNN
-F 2 "Connector_PinSocket_2.54mm:PinSocket_1x06_P2.54mm_Vertical" H 6750 3200 50  0001 C CNN
-F 3 "~" H 6750 3200 50  0001 C CNN
-	1    6750 3200
+P 6750 2950
+F 0 "CN1" H 6778 2926 50  0000 L CNN
+F 1 "To_Amiga" H 6778 2835 50  0000 L CNN
+F 2 "Connector_PinSocket_2.54mm:PinSocket_1x06_P2.54mm_Vertical" H 6750 2950 50  0001 C CNN
+F 3 "~" H 6750 2950 50  0001 C CNN
+	1    6750 2950
 	1    0    0    -1
 $EndComp
 $Comp
-L Connector:Barrel_Jack_MountingPin CN2
+L Connector:Barrel_Jack CN2
 U 1 1 61AA3DB0
 P 2850 3200
 F 0 "CN2" H 2907 3517 50  0000 C CNN
-F 1 "Barrel_Jack_MountingPin" H 2907 3426 50  0000 C CNN
-F 2 "Connector_BarrelJack:BarrelJack_CUI_PJ-102AH_Horizontal" H 2900 3160 50  0001 C CNN
+F 1 "Barrel_Jack" H 2907 3426 50  0000 C CNN
+F 2 "TICK:BarrelJack_Horizontal" H 2900 3160 50  0001 C CNN
 F 3 "~" H 2900 3160 50  0001 C CNN
 	1    2850 3200
@@
 $EndComp
 $Comp
-L 74xGxx:SN74LVC1G14DBV U1
-U 1 1 61AA57DC
-P 5300 3100
-F 0 "U1" H 5400 2950 50  0000 L CNN
-F 1 "74AHCT1G04" H 5400 2850 50  0000 L CNN
-F 2 "Package_TO_SOT_SMD:SOT-23-5" H 5300 2850 50  0001 C CNN
-F 3 "http://www.ti.com/lit/ds/symlink/sn74lvc1g14.pdf" H 5300 3100 50  0001 C CNN
-	1    5300 3100
-	1    0    0    -1
-$EndComp
-$Comp
 L Device:C C1
 U 1 1 61AA66CC
-P 4800 3400
-F 0 "C1" H 4915 3446 50  0000 L CNN
-F 1 "22uF" H 4915 3355 50  0000 L CNN
-F 2 "Capacitor_SMD:C_1206_3216Metric" H 4838 3250 50  0001 C CNN
-F 3 "~" H 4800 3400 50  0001 C CNN
-	1    4800 3400
+P 4150 3400
+F 0 "C1" H 4265 3446 50  0000 L CNN
+F 1 "0.22uF" H 4265 3355 50  0000 L CNN
+F 2 "Capacitor_SMD:C_1206_3216Metric" H 4188 3250 50  0001 C CNN
+F 3 "~" H 4150 3400 50  0001 C CNN
+	1    4150 3400
 	1    0    0    -1
 $EndComp
@@
 P 3800 3100
 F 0 "R1" V 3593 3100 50  0000 C CNN
-F 1 "560" V 3684 3100 50  0000 C CNN
+F 1 "3.3k" V 3684 3100 50  0000 C CNN
 F 2 "Resistor_SMD:R_1206_3216Metric" V 3730 3100 50  0001 C CNN
 F 3 "~" H 3800 3100 50  0001 C CNN
@@
 $EndComp
 $Comp
-L Device:R R2
-U 1 1 61AA6FD0
-P 6050 2500
-F 0 "R2" H 6120 2546 50  0000 L CNN
-F 1 "10k" H 6120 2455 50  0000 L CNN
-F 2 "Resistor_SMD:R_1206_3216Metric" V 5980 2500 50  0001 C CNN
-F 3 "~" H 6050 2500 50  0001 C CNN
-	1    6050 2500
-	1    0    0    -1
-$EndComp
-$Comp
-L Device:D_Zener D1
+L Device:D D1
 U 1 1 61AA7657
-P 4150 3400
-F 0 "D1" V 4104 3480 50  0000 L CNN
-F 1 "MMSZ5225" V 4195 3480 50  0000 L CNN
-F 2 "Diode_SMD:D_SOD-123" H 4150 3400 50  0001 C CNN
-F 3 "~" H 4150 3400 50  0001 C CNN
-	1    4150 3400
+P 4800 3400
+F 0 "D1" V 4754 3480 50  0000 L CNN
+F 1 "1N4148" V 4845 3480 50  0000 L CNN
+F 2 "Diode_SMD:D_SOD-123" H 4800 3400 50  0001 C CNN
+F 3 "~" H 4800 3400 50  0001 C CNN
+	1    4800 3400
 	0    1    1    0
 $EndComp
-NoConn ~ 6550 3000
-NoConn ~ 6550 3400
+NoConn ~ 6550 2750
+NoConn ~ 6550 3150
 Wire Wire Line
-	6550 3500 6550 3900
+	6550 3250 6550 3900
 Wire Wire Line
 	6550 3900 7800 3900
@@
 	1    0    0    -1
 $EndComp
-Wire Wire Line
-	6550 3100 6050 3100
-Text Label 6550 3100 2    50   ~ 0
+Text Label 6550 2850 2    50   ~ 0
 TBASE
 Wire Wire Line
-	6550 3200 6350 3200
-Wire Wire Line
-	6350 3200 6350 3900
+	6350 2950 6350 3900
 $Comp
 L power:GND #PWR?
@@
 	1    0    0    -1
 $EndComp
-NoConn ~ 6550 3300
-Wire Wire Line
-	5300 3300 5300 3900
-Wire Wire Line
-	5300 3900 6350 3900
+NoConn ~ 6550 3050
 Connection ~ 6350 3900
-Wire Wire Line
-	5300 2900 5300 2350
-Wire Wire Line
-	5300 2350 5550 2350
 Connection ~ 7800 2350
-$Comp
-L Device:C C2
-U 1 1 61AAAE02
-P 5550 2500
-F 0 "C2" H 5665 2546 50  0000 L CNN
-F 1 "0.1uF" H 5665 2455 50  0000 L CNN
-F 2 "Capacitor_SMD:C_1206_3216Metric" H 5588 2350 50  0001 C CNN
-F 3 "~" H 5550 2500 50  0001 C CNN
-	1    5550 2500
-	1    0    0    -1
-$EndComp
-Connection ~ 5550 2350
-Wire Wire Line
-	5550 2350 6050 2350
-$Comp
-L power:GND #PWR?
-U 1 1 61AAB60C
-P 5550 2650
-F 0 "#PWR?" H 5550 2400 50  0001 C CNN
-F 1 "GND" H 5555 2477 50  0000 C CNN
-F 2 "" H 5550 2650 50  0001 C CNN
-F 3 "" H 5550 2650 50  0001 C CNN
-	1    5550 2650
-	1    0    0    -1
-$EndComp
-Connection ~ 6050 2350
-Wire Wire Line
-	6050 2350 7800 2350
-Wire Wire Line
-	6050 2650 6050 3100
-Connection ~ 6050 3100
-Wire Wire Line
-	6050 3100 5600 3100
 Wire Wire Line
 	3950 3100 4150 3100
 Wire Wire Line
 	4150 3550 4150 3900
-Connection ~ 5300 3900
 Wire Wire Line
 	4150 3250 4150 3100
@@
 	3150 3900 4150 3900
 Connection ~ 4150 3900
-Wire Wire Line
-	2850 3500 2850 3900
-Wire Wire Line
-	2850 3900 3150 3900
-Connection ~ 3150 3900
 Text Label 3150 3100 0    50   ~ 0
 +9VAC
@@
 Connection ~ 4800 3900
 Wire Wire Line
-	4800 3900 5300 3900
-Wire Wire Line
 	4150 3900 4800 3900
 Wire Wire Line
 	4150 3100 4800 3100
-Text Notes 3600 4150 2    50   ~ 0
-D1 = 3V, 500mw
+$Comp
+L Transistor_BJT:MMBT3904 Q1
+U 1 1 61AED3D3
+P 5300 3100
+F 0 "Q1" H 5491 3146 50  0000 L CNN
+F 1 "MMBT3904" H 5491 3055 50  0000 L CNN
+F 2 "Package_TO_SOT_SMD:SOT-23" H 5500 3025 50  0001 L CIN
+F 3 "https://www.onsemi.com/pub/Collateral/2N3903-D.PDF" H 5300 3100 50  0001 L CNN
+	1    5300 3100
+	1    0    0    -1
+$EndComp
+Wire Wire Line
+	4800 3900 5400 3900
+Wire Wire Line
+	5400 3300 5400 3900
+Connection ~ 5400 3900
+Wire Wire Line
+	5400 3900 6350 3900
+Wire Wire Line
+	5400 2900 5400 2850
+$Comp
+L Device:R R2
+U 1 1 61AEFC1B
+P 5400 2600
+F 0 "R2" V 5193 2600 50  0000 C CNN
+F 1 "4.7k" V 5284 2600 50  0000 C CNN
+F 2 "Resistor_SMD:R_1206_3216Metric" V 5330 2600 50  0001 C CNN
+F 3 "~" H 5400 2600 50  0001 C CNN
+	1    5400 2600
+	-1   0    0    1
+$EndComp
+Wire Wire Line
+	6550 2850 5400 2850
+Connection ~ 5400 2850
+Wire Wire Line
+	5400 2850 5400 2750
+Wire Wire Line
+	5400 2450 5400 2350
+Wire Wire Line
+	5400 2350 7800 2350
+Wire Wire Line
+	6550 2950 6350 2950
 $EndSCHEMATC

Commit message: Add files via upload
Parts:
- R1: value 3.3k -> 4.7k
Changed lines of the file:
@@
 P 3800 3100
 F 0 "R1" V 3593 3100 50  0000 C CNN
-F 1 "3.3k" V 3684 3100 50  0000 C CNN
+F 1 "4.7k" V 3684 3100 50  0000 C CNN
 F 2 "Resistor_SMD:R_1206_3216Metric" V 3730 3100 50  0001 C CNN
 F 3 "~" H 3800 3100 50  0001 C CNN
