File: TICK/TICK_AC/TICK_AC.kicad_pcb (KiCad board)
At the start: 2 copper layers, 33.9 x 19.8 mm, 7 parts, among them CN1 To_Amiga, CN2 Barrel_Jack, Q1 MMBT3904

Commit message: Add files via upload
Parts:
- R1: value 3.3k -> 4.7k
Other:
- board text added: "The time is precious I know"

Commit message: Add files via upload
Other:
- board text added: "9VAC"
- board text added: "The time is precious, I know."
- board text removed: "+9VAC"
- board text removed: "The time is precious I know"
