File: TICK/TICK_OSC/TICK.kicad_pcb (KiCad board)
At the start: 2 copper layers, 37.3 x 27 mm, 10 parts, among them CN1 To_Amiga, U1 74HC4060, U2 74HC73, Y1 3.93216MHz

Commit message: Add files via upload
Parts:
- moved C3 1.95 mm to (149.6, 87.1), turned to 90 degrees
Other:
- board text added: "Original Concept By Michael Schulz"
- board text added: "Y1 = 3.2768MHz for 50Hz 3.93216MHz for 60Hz"
