File: TICK/TICK_OSC/TICK.sch (KiCad schematic (older format))
At the start: 10 parts, among them CN1 To_Amiga, U1 74HC4060, U2 74HC73, Y1 3.93216MHz

Commit message: Add files via upload
Other:
- note added: "Y1 =\n3.2768 MHz for PAL 50Hz TICK\n3.93216MHz for NTSC 60Hz TICK"
Changed lines of the file:
@@
 Wire Wire Line
 	3350 3700 3175 3700
+Text Notes 1925 5275 0    79   ~ 0
+Y1 =\n3.2768 MHz for PAL 50Hz TICK\n3.93216MHz for NTSC 60Hz TICK
 $EndSCHEMATC
